File: dipconn.sch (KiCad schematic (older format))
At the start: 6 parts, among them J3 idc2k, J4 dip2k, J5 idc32k, J6 dip32k

Commit message: renamed to emurom
Parts:
- J3: footprint romdev:conn2k -> emurom:conn2k
- J5: footprint romdev:conn32k -> emurom:conn32k
Changed lines of the file:
@@
 F 0 "J5" H 7750 3367 50  0000 C CNN
 F 1 "idc32k" H 7750 3276 50  0000 C CNN
-F 2 "romdev:conn32k" H 7700 2550 50  0001 C CNN
+F 2 "emurom:conn32k" H 7700 2550 50  0001 C CNN
 F 3 "~" H 7700 2550 50  0001 C CNN
 	1    7700 2550
@@
 F 0 "J3" H 4250 3367 50  0000 C CNN
 F 1 "idc2k" H 4250 3276 50  0000 C CNN
-F 2 "romdev:conn2k" H 4200 2650 50  0001 C CNN
+F 2 "emurom:conn2k" H 4200 2650 50  0001 C CNN
 F 3 "~" H 4200 2650 50  0001 C CNN
 	1    4200 2650
