File: emurom.sch (KiCad schematic (older format))
At the start: 41 parts, among them J1 AVR-ISP, J2 USB_B_Micro, J7 SYSRST, U1 ATmega328P-AU, U10 conn2k, U11 conn32k, U2 mcp2221, U3 74HCT157, U4 74HCT595, U5 74HCT595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

Commit message: renamed to emurom
Parts:
- U1: symbol romdev:ATmega328P-AU -> emurom:ATmega328P-AU
- U10: footprint romdev:conn2k -> emurom:conn2k; symbol romdev:conn2k -> emurom:conn2k
- U11: footprint romdev:conn32k -> emurom:conn32k; symbol romdev:conn32k -> emurom:conn32k
- U2: symbol romdev:mcp2221 -> emurom:mcp2221
- U6: symbol romdev:sram_um61512ak -> emurom:sram_um61512ak
Changed lines of the file:
@@
 $EndComp
 $Comp
-L romdev:sram_um61512ak U6
+L emurom:sram_um61512ak U6
 U 1 1 5EC358D5
 P 5550 2150
@@
 $EndComp
 $Comp
-L romdev:mcp2221 U2
+L emurom:mcp2221 U2
 U 1 1 5EC41AB3
 P 2700 5500
@@
 	2800 1750 3150 1750
 $Comp
-L romdev:ATmega328P-AU U1
+L emurom:ATmega328P-AU U1
 U 1 1 5ED09330
 P 2200 2950
@@
 A[0..15]
 $Comp
-L romdev:conn32k U11
+L emurom:conn32k U11
 U 1 1 5FAB03BB
 P 9500 5050
 F 0 "U11" H 9600 5950 50  0000 C CNN
 F 1 "conn32k" V 9500 5100 50  0000 C CNN
-F 2 "romdev:conn32k" H 9500 5050 50  0001 C CNN
+F 2 "emurom:conn32k" H 9500 5050 50  0001 C CNN
 F 3 "" H 9500 5050 50  0001 C CNN
 	1    9500 5050
@@
 $EndSheet
 $Comp
-L romdev:conn2k U10
+L emurom:conn2k U10
 U 1 1 5FBD48AD
 P 9500 2600
 F 0 "U10" H 9600 3350 50  0000 C CNN
 F 1 "conn2k" V 9500 2600 50  0000 C CNN
-F 2 "romdev:conn2k" H 9500 2450 50  0001 C CNN
+F 2 "emurom:conn2k" H 9500 2450 50  0001 C CNN
 F 3 "" H 9500 2450 50  0001 C CNN
 	1    9500 2600
